File: pcb/Empyrean.sch (KiCad schematic (older format))
At the start: 40 parts, among them J1 FCI 10118194-0001LF, J2 Harwin M50-3500542, J3 SPI, J4 CONN_01X15, J5 CONN_01X15, Q1 2N7002TQ, U1 LP2985, U2 ATSAMD21GxA, X1 ECS-.327-12.5-34B-TR

Commit message: Set proper rev on documentation
Parts:
- C1: symbol Empyrean-rescue:C -> EtherkitKicadLibrary:C; MPN (none) -> CC0603KRX7R9BB472
- C10, C11, C12, C6, C8: symbol Empyrean-rescue:C -> EtherkitKicadLibrary:C; MPN (none) -> CC0603KRX7R9BB104
- C2, C7: symbol Empyrean-rescue:C -> EtherkitKicadLibrary:C; MPN (none) -> CC0603MRX5R5BB106
- C3, C9: symbol Empyrean-rescue:C -> EtherkitKicadLibrary:C; MPN (none) -> CC0603KRX5R8BB105
- C4, C5: symbol Empyrean-rescue:C -> EtherkitKicadLibrary:C; MPN (none) -> GCM1885C1H150JA16D
- D1: symbol Empyrean-rescue:LED -> EtherkitKicadLibrary:LED; MPN (none) -> LTST-C170KGKT; URL (none) -> https://www.mouser.com/ProductDetail/Lite-On/LTST-C170KGKT?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
- D2: symbol Empyrean-rescue:LED -> EtherkitKicadLibrary:LED; MPN (none) -> LTST-C170KSKT; URL (none) -> https://www.mouser.com/ProductDetail/Lite-On/LTST-C170KSKT?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
- D3: symbol Empyrean-rescue:LED -> EtherkitKicadLibrary:LED; MPN (none) -> LTST-C170TBKT; URL (none) -> https://www.mouser.com/ProductDetail/Lite-On/LTST-C170TBKT?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
- D4: symbol Empyrean-rescue:LED -> EtherkitKicadLibrary:LED; MPN (none) -> LTST-C170KRKT; URL (none) -> https://www.mouser.com/ProductDetail/Lite-On/LTST-C170KRKT?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
- F1: MPN (none) -> 0ZCH0050FF2G; URL (none) -> https://www.mouser.com/ProductDetail/Bel-Fuse/0ZCH0050FF2G?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
- J1: MPN (none) -> 10118194-0001LF; URL (none) -> https://www.mouser.com/ProductDetail/Amphenol-FCI/10118194-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
- J2: symbol Empyrean-rescue:CONN_02X05 -> EtherkitKicadLibrary:CONN_02X05
- J3: symbol Empyrean-rescue:CONN_01X03 -> Connector_Generic:Conn_01x03
- J4, J5: symbol Empyrean-rescue:CONN_01X15 -> Connector_Generic:Conn_01x15
- JP1, JP2: symbol Empyrean-rescue:JUMPER-NC-EtherkitKicadLibrary -> EtherkitKicadLibrary:JUMPER-NC
- L1: symbol Empyrean-rescue:L -> EtherkitKicadLibrary:L; MPN (none) -> MLF1608E100JT000
- Q1: symbol Empyrean-rescue:MOS_N -> EtherkitKicadLibrary:MOS_N; MPN (none) -> 2N7002TQ-7-F; URL (none) -> https://www.mouser.com/ProductDetail/Diodes-Incorporated/2N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
- R1, R3, R4, R5, R6, R8: symbol Empyrean-rescue:R -> EtherkitKicadLibrary:R; MPN (none) -> RC0603FR-07330RL
- R2: symbol Empyrean-rescue:R -> EtherkitKicadLibrary:R; MPN (none) -> RC0603FR-071ML
- R7: symbol Empyrean-rescue:R -> EtherkitKicadLibrary:R; MPN (none) -> RC0603JR-0710KL
- S1: symbol Empyrean-rescue:PUSHBUTTON -> EtherkitKicadLibrary:PUSHBUTTON; MPN (none) -> SKQMASE010; URL (none) -> https://www.mouser.com/ProductDetail/ALPS/SKQMASE010?qs=%2F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
- U1: symbol Empyrean-rescue:LP2985 -> EtherkitKicadLibrary:LP2985; MPN (none) -> LP2985-33DBVR; URL (none) -> https://www.mouser.com/ProductDetail/Texas-Instruments/LP29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
- U2: symbol Empyrean-rescue:ATSAMD21G18A -> EtherkitKicadLibrary:ATSAMD21G18A; MPN (none) -> ATSAMD21G18A-AUT; URL (none) -> https://www.mouser.com/ProductDetail/Microchip-Technology/A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
- VR1, VR2: symbol Empyrean-rescue:VR -> EtherkitKicadLibrary:VR; MPN (none) -> CG0603MLC-05E; URL (none) -> https://www.mouser.com/ProductDetail/Bourns/CG0603MLC-05E?q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
- X1: symbol Empyrean-rescue:CRYSTAL -> EtherkitKicadLibrary:CRYSTAL; MPN (none) -> ECS-.327-12.534B-TR; URL (none) -> https://www.mouser.com/ProductDetail/ECS/ECS-327-125-34B-TR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
