File: pcb/_autosave-Empyrean.kicad_pcb (KiCad board)
At the start: 2 copper layers, 18.3 x 45.6 mm, 46 parts, among them J1 FCI 10118194-0001LF, J2 Harwin M50-3500542, J3 SPI, J4 CONN_01X15, J5 CONN_01X15, Q1 DMG1012T-7, U1 LP2985, U2 ATSAMD21GxA, X1 ECS-.327-12.5-34B-TR

Commit message: Set proper rev on documentation
Parts:
- Q1: value DMG1012T-7 -> 2N7002TQ-7-F
Changed lines of the file:
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@@
     (last_trace_width 0.2)
     (trace_clearance 0.13)
-    (zone_clearance 0.16)
+    (zone_clearance 0.14)
     (zone_45_only yes)
     (trace_min 0.16)
@@
       (effects (font (size 0.6 0.6) (thickness 0.1)))
     )
-    (fp_text value DMG1012T-7 (at 0 0) (layer F.SilkS) hide
+    (fp_text value 2N7002TQ-7-F (at 0 0) (layer F.SilkS) hide
       (effects (font (size 0.6 0.6) (thickness 0.1)))
     )
@@
   )
   (zone (net 1) (net_name GND) (layer F.Cu) (hatch edge 0.508)
-    (connect_pads (clearance 0.16))
-    (min_thickness 0.16)
+    (connect_pads (clearance 0.14))
+    (min_thickness 0.14)
     (fill yes (arc_segments 16) (thermal_gap 0.16) (thermal_bridge_width 0.22) (smoothing chamfer))
     (polygon
